Commit message: Added turtlebot2 files to master

File: robots/katka.urdf.xacro (robot description, xacro)
@@ -6,4 +6,5 @@
 -->
 <robot name="turtlebot" xmlns:xacro="http://ros.org/wiki/xacro">
+  <!--<xacro:include filename="$(find turtlebot_description)/urdf/turtlebot_library.urdf.xacro" />-->
   <xacro:include filename="$(find turtlebot_description)/urdf/turtlebot_library.urdf.xacro" />
   <xacro:include filename="$(find icclab_turtlebot)/sensors/rplidar.urdf.xacro" />
@@ -12,5 +13,6 @@
   <sensor_kinect  parent="base_link"/>
   <xacro:rplidar name="rplidar" parent="base_link" ros_topic="scan" update_rate="5" ray_count="1040" min_angle="0" max_angle="360">
-    <origin xyz="-0.1 0 0.420" rpy="3.1415 0 1.5707"/>
+    <!--<origin xyz="-0.1 0 0.420" rpy="3.1415 0 1.5707"/>-->
+    <origin xyz="0.1 0 0.420" rpy="3.1415 0 3.1415"/>
   </xacro:rplidar>
 </robot>

File: robots/turtlebot.urdf.xacro (robot description, xacro)
@@ -12,5 +12,5 @@
   <sensor_kinect  parent="base_link"/>
   <xacro:rplidar name="rplidar" parent="base_link" ros_topic="scan" update_rate="5" ray_count="1040" min_angle="0" max_angle="360">
-    <origin xyz="0.1 0 0.420" rpy="0 0 0"/>
+    <origin xyz="0.1 0 0.35" rpy="0 0 0"/>
   </xacro:rplidar>
 </robot>
