Commit message: Edited urdf lidar to be at physical position, costmap now gets data from both kinect and rplidar, amcl_demo works amcl_demo.launch + minimal_with_rplidar.launch

File: robots/turtlebot.urdf.xacro (robot description, xacro)
@@ -12,5 +12,5 @@
   <sensor_kinect  parent="base_link"/>
   <xacro:rplidar name="rplidar" parent="base_link" ros_topic="scan" update_rate="5" ray_count="1040" min_angle="0" max_angle="360">
-    <origin xyz="0.1 0 0.420" rpy="3.1415 0 3.1415"/>
+    <origin xyz="0.1 0 0.33" rpy="3.1415 0 3.1415"/> <!-- laserscan topic is at approx physical height -->
   </xacro:rplidar>
 </robot>
